File: Disk & Floppy.kicad_sch (KiCad schematic)
At the start: 33 parts, among them J12 External HDD, J13 FDD Power, J7 Internal FDD, U18 74LS74, U19 74LS244, U20 74LS245, U21 74LS74, U22 74LS05, U37 DMA, U38 WD1772, X1 8.010613MHz

Commit message: motherboard: Fixed a pile of resistor network issues, and concluded initial routing of the CPU and audio amp passives
Parts:
- RN13, RN14, RN15: symbol Device:R_Pack04 -> dragonmux:R_Pack04_OddEven
Connections:
- net HDA0: now also RN15.5 (R4.2); no longer RN15.3 (R3.1)
- net HDR/~{W}: now also RN15.7 (R2.2); no longer RN15.4 (R4.1)
- net ~{HDACK}: now also RN15.3 (R3.1); no longer RN15.2 (R2.1)
- net at U19.12 (O3a): now also RN15.8 (R1.2); no longer RN15.5 (R4.2)
- net at U19.3 (O3b): now also RN15.4 (R4.1); no longer RN15.7 (R2.2)
- net at U19.5 (O2b): now also RN15.2 (R2.1); no longer RN15.8 (R1.2)
- net at U20.2 (A0): now also RN14.8 (R1.2); no longer RN14.5 (R4.2)
- net at U20.4 (A2): now also RN14.4 (R4.1); no longer RN14.7 (R2.2)
- net at U20.5 (A3): now also RN14.2 (R2.1); no longer RN14.8 (R1.2)
- net at U20.6 (A4): now also RN13.8 (R1.2); no longer RN13.5 (R4.2)
- net at U20.8 (A6): now also RN13.4 (R4.1); no longer RN13.7 (R2.2)
- net at U20.9 (A7): now also RN13.2 (R2.1); no longer RN13.8 (R1.2)
- net at J12.7: now also RN13.3 (R3.1); no longer RN13.2 (R2.1)
- net at J12.6: now also RN13.5 (R4.2); no longer RN13.3 (R3.1)
- net at J12.5: now also RN13.7 (R2.2); no longer RN13.4 (R4.1)
- net at J12.1: now also RN14.7 (R2.2); no longer RN14.4 (R4.1)
- net at J12.2: now also RN14.5 (R4.2); no longer RN14.3 (R3.1)
- net at J12.3: now also RN14.3 (R3.1); no longer RN14.2 (R2.1)
Changed lines of the file:
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@@
 	)
 	(symbol
-		(lib_id "Device:R_Pack04")
+		(lib_id "dragonmux:R_Pack04_OddEven")
 		(at 119.38 60.96 90)
 		(unit 1)
@@
 		)
 		(property "Description" "4 resistor network, parallel topology"
-			(at 119.38 60.96 0)
+			(at 132.08 62.23 0)
 			(effects
 				(font
@@
 	)
 	(symbol
-		(lib_id "Device:R_Pack04")
+		(lib_id "dragonmux:R_Pack04_OddEven")
 		(at 111.76 127 90)
 		(unit 1)
@@
 		)
 		(property "Description" "4 resistor network, parallel topology"
-			(at 111.76 127 0)
+			(at 124.46 128.27 0)
 			(effects
 				(font
@@
 	)
 	(symbol
-		(lib_id "Device:R_Pack04")
+		(lib_id "dragonmux:R_Pack04_OddEven")
 		(at 111.76 116.84 90)
 		(unit 1)
@@
 		)
 		(property "Description" "4 resistor network, parallel topology"
-			(at 111.76 116.84 0)
-			(effects
-				(font
+			(at 124.46 118.11 0)
+			(effects
+				(font

Commit message: motherboard: Added packaging and ordering information for many of the 7400 logic parts and the DACs
Parts:
- U18, U21: value 74LS74 -> 74HC74; footprint (none) -> rhais_package-smd:SO-14_3.9x8.65mm_P1.27mm; MFR (none) -> Nexperia; MPN (none) -> 74HC74D,653; OC_FARNELL (none) -> 1201317
- U19: value 74LS244 -> 74HC244; footprint (none) -> Package_SO:SO-20_12.8x7.5mm_P1.27mm; MFR (none) -> Nexperia; MPN (none) -> 74HC244D,653; OC_FARNELL (none) -> 1201322
- U20: value 74LS245 -> 74HC245; footprint (none) -> Package_SO:SO-20_12.8x7.5mm_P1.27mm; MFR (none) -> Nexperia; MPN (none) -> 74HC245D,653; OC_FARNELL (none) -> 1201324
- U22: value 74LS05 -> 74HS05
