File: Serial Interface.kicad_sch (KiCad schematic)
At the start: 10 parts, among them U11 ADM232A, U12 ADM232A

Commit message: motherboard: Added more footprints for parts and refined the serial comms section further
Parts:
- added C116, C117: 100n, rhais_rcl:C0603, symbol Device:C_Small
- U11, U12: footprint (none) -> rhais_package-smd:SO-16_3.9x9.9mm_P1.27mm
Connections:
- net +5V: now also C116.1, C117.1
- net GND: now also U12.11 (T1IN), C116.2, C117.2
- net RS232_DIR: now also U12.7 (T2OUT); no longer U12.14 (T1OUT)
- net UART_DIR: now also U12.10 (T2IN); no longer U12.11 (T1IN)
- no-connect marks 0 -> 1
